File: Hardware/Stealthburner_Toolhead_PCB.kicad_pcb (KiCad board)
At the start: 4 copper layers, 47 x 43 mm, 144 parts, among them J1 Conn_01x02, J10 Conn_01x05, J11 Conn_01x04, J12 Conn_01x04, J2 Conn_01x03, J3 TestPoint, J4 Conn_01x02, J5 Conn_01x03, J6 Conn_01x02, J7 Conn_01x05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

Commit message: V2.1 Release
将1.25mm连接器替换为2.0mm
使用MicroUSB母座作为USB连接器
修改PCB尺寸

Replace Molex PicoBlade Connector with PH2.0 Connector
Replace USB connector with Micro USB port
Modified PCB size
Parts:
- removed kibuzzard-62BB2432: G***, kibuzzard-62BB2432
- removed kibuzzard-62BB2448: G***, kibuzzard-62BB2448
- removed kibuzzard-62BB2459: G***, kibuzzard-62BB2459
- added G***: LOGO, LOGO, F.Cu at (144.5, 113.8)
- added kibuzzard-63148E7F: G***, kibuzzard-63148E7F, B.Cu at (133.0, 112.0)
- added kibuzzard-63148E89: G***, kibuzzard-63148E89, B.Cu at (135.1, 112.0)
- added kibuzzard-63148E96: G***, kibuzzard-63148E96, B.Cu at (131.0, 112.0)
- G***, kibuzzard-62BB2226, kibuzzard-62BB2232: moved to B.Cu
- J10, J7: footprint 1_Library:Molex_PicoBlade_53047-0510_1x05_P1.25mm_Vertical -> Connector_Molex:Molex_PicoBlade_53261-0571_1x05-1MP_P1.25mm_Horizontal
- J2, J8: footprint 1_Library:Molex_PicoBlade_53047-0310_1x03_P1.25mm_Vertical -> Connector_JST:JST_PH_B3B-PH-K_1x03_P2.00mm_Vertical
- J4, J6: footprint 1_Library:Molex_PicoBlade_53047-0210_1x02_P1.25mm_Vertical -> Connector_JST:JST_PH_B2B-PH-K_1x02_P2.00mm_Vertical
- J5: value Conn_01x03 -> USB_B_Micro; footprint 1_Library:Molex_PicoBlade_53047-0310_1x03_P1.25mm_Vertical -> Connector_USB:USB_Micro-B_Molex_47346-0001
- U12: value TMC2209-LA-T -> QFN28_5X5_3X8_EPAD_TRI
- U4: value W25Q16JVUXIQ -> W25Q16JVUXIQ_WIN
- moved G*** 13.7 mm to (143.0, 115.2), turned to -90 degrees
- moved J8 12.0 mm to (135.0, 110.5), turned to 180 degrees
- moved R18 8.79 mm to (104.7, 108.3), turned to 0 degrees
- moved J5 7.46 mm to (144.2, 121.0)
- moved R13 7.28 mm to (106.5, 108.3), turned to 180 degrees
- moved R8 6.00 mm to (139.2, 115.8), turned to -90 degrees
- moved R20 5.87 mm to (108.4, 107.3), turned to 0 degrees
- moved J10 5.54 mm to (102.8, 102.3), turned to -90 degrees
- moved Q2 5.53 mm to (102.2, 102.9), turned to 90 degrees
- moved kibuzzard-62BB2232 4.93 mm to (121.4, 97.2)
- moved R10 4.72 mm to (140.1, 115.8), turned to 90 degrees
- moved J12 4.16 mm to (139.3, 132.0)
- moved D3 4.12 mm to (102.2, 110.8), turned to 0 degrees
- moved D4 4.10 mm to (102.2, 109.5), turned to 0 degrees
- moved Q1 4.10 mm to (102.2, 113.5)
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Connections:
- J10 pad 1: Net-(J10-Pad1) -> /FAN2_DET
- J10 pad 2: GND -> Net-(D5-Pad2)
- J10 pad 4: Net-(D5-Pad2) -> GND
- J10 pad 5: /FAN2_DET -> Net-(J10-Pad5)
- J5 pad 1: GND -> unconnected-(J5-Pad1)
- J7 pad 1: Net-(J7-Pad1) -> /FAN1_DET
- J7 pad 2: GND -> Net-(D3-Pad2)
- J7 pad 4: Net-(D3-Pad2) -> GND
- J7 pad 5: /FAN1_DET -> Net-(J7-Pad5)
- JP1 pad 2: Net-(J7-Pad1) -> Net-(J7-Pad5)
- JP2 pad 2: Net-(J10-Pad1) -> Net-(J10-Pad5)
- R10 pad 1: Net-(J5-Pad2) -> Net-(J5-Pad3)
- R8 pad 2: Net-(J5-Pad3) -> Net-(J5-Pad2)
- U5 pad 1: /D- -> /D+
- U5 pad 3: /D+ -> /D-
- U5 pad 4: Net-(R10-Pad2) -> Net-(R8-Pad1)
- U5 pad 6: Net-(R8-Pad1) -> Net-(R10-Pad2)
Routing:
- net Net-(J8-Pad2): track 2.32 -> 13.5 mm
- net +5V: track 63.5 -> 52.4 mm, vias 4 -> 3
- net +12V: track 67.8 -> 57.9 mm, vias 11 -> 9
- net /FAN1_PWM: track 11.2 -> 3.45 mm
- net +3V3: track 193.5 -> 187.2 mm, vias 19 -> 22
- net /D-: track 29.1 -> 34.9 mm
- net /D+: track 30.0 -> 35.0 mm
- net /FAN2_PWM: track 9.09 -> 5.37 mm
- net Net-(J5-Pad2): track 3.49 -> 7.16 mm
- net Net-(J7-Pad5): track 0.00 -> 3.67 mm, vias 0 -> 1
- net Net-(D5-Pad1): track 7.03 -> 3.37 mm
- net Net-(J10-Pad5): track 0.00 -> 3.61 mm, vias 0 -> 1
- net Net-(J5-Pad3): track 3.39 -> 6.81 mm
- net Net-(C17-Pad1): track 4.62 -> 7.19 mm
- net Net-(J10-Pad3): track 5.10 -> 3.24 mm, vias 0 -> 1
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- added copper zone on B.Cu, net +3V3
- removed copper zone on In1.Cu, net /D+
- removed copper zone on F.Cu, net /E-A2
- removed copper zone on F.Cu, net /E-B2
Other:
- board size 47 x 43 mm -> 47 x 39.5 mm
- board text added: "3"
- board text added: "Bot"
- board text added: "In1"
- board text added: "In2"
- board text added: "Top"
- board text added: "V2.1"
- board text removed: "D+"
- board text removed: "D-"
- board text removed: "Designed by"
- board text removed: "V1.2"
