File: Hardware/Stealthburner_Toolhead_PCB.kicad_sch (KiCad schematic)
At the start: 111 parts, among them J1 Conn_01x02, J10 Conn_01x05, J11 Conn_01x04, J12 Conn_01x04, J2 Conn_01x03, J3 TestPoint, J4 Conn_01x02, J5 Conn_01x03, J6 Conn_01x02, J7 Conn_01x05, J8 Conn_01x03, J9 Conn_01x02, Q1 AO3400A, Q2 AO3400A, Q3 WSD4038DN, U1 BL9342, U10 74LVC1G32, U11 TMC2209-LA-T, U12 MAX31865xTP, U13 ADXL343, U14 SHT31-DIS, U2 ME6209A50M3G, U3 ME6209A33M3G, U4 W25Q16JVUXIQ, U5 USBLC6-2SC6, U6 74LVC2G17, U7 RP2040, U8 74LVC2G17, U9 SHT20, Y1 CSTNE12M0

Commit message: 1
Parts:
- C35: renamed from C?; footprint (none) -> Capacitor_SMD:C_0603_1608Metric
- gave numbers to parts that had none: 2
- renumbered C35 to C36
Changed lines of the file:
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@@
   (symbol (lib_id "Device:C") (at 668.02 145.415 0) (unit 1)
     (in_bom no) (on_board no)
-    (property "Reference" "C35" (id 0) (at 668.02 142.875 0)
+    (property "Reference" "C36" (id 0) (at 668.02 142.875 0)
       (effects (font (size 1.27 1.27)) (justify left))
     )
@@
   (symbol (lib_id "Device:C_Small") (at 389.89 235.585 0) (unit 1)
     (in_bom yes) (on_board yes)
-    (property "Reference" "C?" (id 0) (at 391.795 234.315 0)
+    (property "Reference" "C35" (id 0) (at 391.795 234.315 0)
       (effects (font (size 1.27 1.27)) (justify left))
     )
@@
       (effects (font (size 1.27 1.27)) (justify left))
     )
-    (property "Footprint" "" (id 2) (at 389.89 235.585 0)
+    (property "Footprint" "Capacitor_SMD:C_0603_1608Metric" (id 2) (at 389.89 235.585 0)
       (effects (font (size 1.27 1.27)) hide)
     )
@@
   (symbol (lib_id "Motor:Fan_3pin") (at 697.865 229.87 180) (unit 1)
     (in_bom no) (on_board no) (fields_autoplaced)
-    (property "Reference" "M?" (id 0) (at 693.42 226.0599 0)
+    (property "Reference" "M1" (id 0) (at 693.42 226.0599 0)
       (effects (font (size 1.27 1.27)) (justify left) hide)
     )
@@
   (symbol (lib_id "Device:Thermistor_NTC_4Wire") (at 684.53 90.17 0) (unit 1)
     (in_bom no) (on_board no) (fields_autoplaced)
-    (property "Reference" "TH?" (id 0) (at 687.705 88.8999 0)
+    (property "Reference" "TH1" (id 0) (at 687.705 88.8999 0)
       (effects (font (size 1.27 1.27)) (justify left) hide)
     )
@@
       (reference "C34") (unit 1) (value "100nF") (footprint "Capacitor_SMD:C_0402_1005Metric")
     )
-    (path "/2f7e3f31-0eda-4661-8ba1-38529ac401db"
-      (reference "C35") (unit 1) (value "100nF") (footprint "Capacitor_SMD:C_0402_1005Metric")
-    )
     (path "/3583a4cb-81b7-48d3-9502-ae19382dc637"
-      (reference "C?") (unit 1) (value "100nF/1uF") (footprint "")
+      (reference "C35") (unit 1) (value "100nF/1uF") (footprint "Capacitor_SMD:C_0603_1608Metric")
+    )
+    (path "/2f7e3f31-0eda-4661-8ba1-38529ac401db"
+      (reference "C36") (unit 1) (value "100nF") (footprint "Capacitor_SMD:C_0402_1005Metric")
     )
     (path "/97fa61a9-5012-4aa2-b1b7-84df384d12c0"
@@
     )
     (path "/c60eec6c-3a0c-4898-be6f-9ab9a8ddeb52"
-      (reference "M?") (unit 1) (value "Fan_3pin") (footprint "")
+      (reference "M1") (unit 1) (value "Fan_3pin") (footprint "")
     )
     (path "/f1d25ee1-e9b3-414d-9ace-e56b7bdd884f"
@@
     )
     (path "/c6b12edc-5bef-41b2-a740-199254408d73"
-      (reference "TH?") (unit 1) (value "Thermistor_NTC_4Wire") (footprint "")
+      (reference "TH1") (unit 1) (value "Thermistor_NTC_4Wire") (footprint "")
     )
     (path "/fb699279-56d8-4959-abfa-353129baa864"

Commit message: 1
Other:
- note added: "Unused"
- moved on the sheet: C28, C36, R29, U14, U9

Commit message: 1
Parts:
- added R22, R23: 10K, Resistor_SMD:R_0402_1005Metric, symbol Device:R
- C1: value 22uF -> 22uF/35V
- L1: value 15uH -> 6.2uH
- renumbered C36 to C26, C26 to C27, C27 to C28, C28 to C29, C29 to C30, C30 to C31, C31 to C32, C32 to C33, C33 to C34, C34 to C35, C35 to C36, R29 to R21, R21 to R24, R22 to R25, R23 to R26, R24 to R27, R25 to R28, R26 to R29, R27 to R30, R28 to R31, U14 to U10, U10 to U11, U11 to U12, U12 to U13, U13 to U14
Connections:
- net +3V3: now also R22.1, R23.1
- net IIC0_SCL: now also R23.2
- net IIC0_SDA: now also R22.2
Other:
- moved on the sheet: C1, C29, U9

Commit message: V1.1 Release
* Add a TVS for TMC2209
* Replaced SHT21 with Si7021
Parts:
- removed U9: SHT20, 1_Library:SHT20, symbol 1_Lib:SHT20
- added D7: SMF28A, Diode_SMD:D_SOD-123F, symbol Diode:SMF28A
- added JP3, JP4: SolderJumper_2_Open, 1_Library:SolderJumper-2_P1.3mm_Open_TrianglePad1.0x1.5mm, symbol Jumper:SolderJumper_2_Open
- added U9: Si7021-A20, Package_DFN_QFN:DFN-6-1EP_3x3mm_P1mm_EP1.5x2.4mm, symbol Sensor_Humidity:Si7021-A20
- D1: value CUS10S30 -> SS14L
- J11: footprint Connector_Molex:Molex_PicoBlade_53261-0471_1x04-1MP_P1.25mm_Horizontal -> 1_Library:JST_PH_S4B-PH-SM4-TB_1x04-1MP_P2.00mm_Horizontal
- R2: value 124K -> 309K
- R3: value 8.87K -> 22.1K
- U1: value BL9342 -> LMR54410
- renumbered JP3 to JP5
Connections:
- net +24V: now also D7.1 (A1)
- net +3V3: now also U9.5 (VDD)
- net FORCE+: now also JP3.2 (B)
- net FORCE-: now also JP4.1 (A)
- net GND: now also D7.2 (A2), U9.2 (GND), U9.7 (PAD)
- net IIC0_SCL: now also U9.6 (SCL)
- net IIC0_SDA: now also U9.1 (SDA)
- net RTDIN+: now also JP3.1 (A)
- net RTDIN-: now also JP4.2 (B)
- no-connect marks 10 -> 11
Other:
- note added: "CHIP | CIN |CBOOST | L | D | RFBt | RFBb LMR14010 | 4.7u |0.1u | 33u | | 301K | 20.5K LMR54410 | 22u |0.1u | 15u | NC | 309K | 22.1K LMR14006Y | 4.7u |0.1u | 18u | | 88.7K | 6.04K"
- note removed: "CHIP | CIN |CBOOST | L | D | RFBt | RFBb BL9342 | 4.7u |0.1u | 6.2u | | 124K | 8.87K LMR54410 | 22u |0.1u | 15u | NC | 309K | 22.1K LMR14006Y | 4.7u |0.1u | 18u | | 88.7K | 6.04K"
- moved on the sheet: C29, J11

Commit message: V1.2 Release
*Changelog*

* 略微修改PCB尺寸与原件布局，防止板子与打印件干涉
* 删除了温度传感器周围的铺铜
* 修复一些小bug
Parts:
- J10, J7: symbol Connector_Generic_MountingPin:Conn_01x05_MountingPin -> Connector_Generic:Conn_01x05
- J2, J5, J8: symbol Connector_Generic_MountingPin:Conn_01x03_MountingPin -> Connector_Generic:Conn_01x03
- J4, J6: symbol Connector_Generic_MountingPin:Conn_01x02_MountingPin -> Connector_Generic:Conn_01x02
Connections:
- net GND: no longer J10.MP (MountPin), J2.MP (MountPin), J4.MP (MountPin), J6.MP (MountPin), J7.MP (MountPin), J8.MP (MountPin)
Other:
- note added: "height of C32 <= 7mm"

Commit message: V2.1 Release
将1.25mm连接器替换为2.0mm
使用MicroUSB母座作为USB连接器
修改PCB尺寸

Replace Molex PicoBlade Connector with PH2.0 Connector
Replace USB connector with Micro USB port
Modified PCB size
Parts:
- removed J5: Conn_01x03, 1_Library:Molex_PicoBlade_53047-0310_1x03_P1.25mm_Vertical, symbol Connector_Generic:Conn_01x03
- added J5: USB_B_Micro, Connector_USB:USB_Micro-B_Molex_47346-0001, symbol Connector:USB_B_Micro
- J10, J7: footprint 1_Library:Molex_PicoBlade_53047-0510_1x05_P1.25mm_Vertical -> Connector_Molex:Molex_PicoBlade_53261-0571_1x05-1MP_P1.25mm_Horizontal; symbol Connector_Generic:Conn_01x05 -> Connector_Generic_MountingPin:Conn_01x05_MountingPin
- J2, J8: footprint 1_Library:Molex_PicoBlade_53047-0310_1x03_P1.25mm_Vertical -> Connector_JST:JST_PH_B3B-PH-K_1x03_P2.00mm_Vertical
- J4, J6: footprint 1_Library:Molex_PicoBlade_53047-0210_1x02_P1.25mm_Vertical -> Connector_JST:JST_PH_B2B-PH-K_1x02_P2.00mm_Vertical
Connections:
- net D+: now also U5.1 (I/O1); no longer U5.3 (I/O2)
- net D-: now also U5.3 (I/O2); no longer U5.1 (I/O1)
- net FAN1_DET: now also J7.1 (Pin_1); no longer J7.5 (Pin_5)
- net FAN2_DET: now also J10.1 (Pin_1); no longer J10.5 (Pin_5)
- net GND: now also J10.4 (Pin_4), J10.MP (MountPin), J7.4 (Pin_4), J7.MP (MountPin), J5.5 (GND), J5.6 (Shield); no longer J10.2 (Pin_2), J7.2 (Pin_2)
- net at D3.2 (A): now also J7.2 (Pin_2); no longer J7.4 (Pin_4)
- net at R8.1: now also U5.4 (I/O2); no longer U5.6 (I/O1)
- net at R8.2: now also J5.2 (D-)
- net at JP1.2 (C): now also J7.5 (Pin_5); no longer J7.1 (Pin_1)
- net at JP2.2 (C): now also J10.5 (Pin_5); no longer J10.1 (Pin_1)
- net at D5.2 (A): now also J10.2 (Pin_2); no longer J10.4 (Pin_4)
- net at R10.1: now also J5.3 (D+)
- net at R10.2: now also U5.6 (I/O1); no longer U5.4 (I/O2)
- no-connect marks 11 -> 13
Other:
- moved on the sheet: R10, R8, U5
